Commit message: First working inverse kinematics code

File: code/goat_arm.urdf (robot description, URDF)
Before this commit: robot robot_arm, 6 links, 5 joints
Links:
- removed link base_rotator
- added link fingertips; visual cylinder length=0.05 radius=2.0
- added link rotator; visual cylinder length=3.7 radius=2.0
- link upper_arm: geometry visual cylinder length=12.0 radius=2.0
Joints:
- added joint last_joint: type revolute, parent fingers, child fingertips, origin xyz=0 0 7.0 rpy=0 0 0, axis 0 0 1, limit lower=-0.01 upper=0.01
- joint base_joint: axis 0 0 -1 -> 0 0 1; child base_rotator -> rotator; origin xyz=0 0 15.15 rpy=0 0 0 -> xyz=0 0 13.3 rpy=0 0 0
- joint elbow_joint: limit lower=-1.92 upper=1.92 -> lower=-1.57 upper=1.57; origin xyz=0 0 31.3 rpy=0 0 0 -> xyz=0 0 12.0 rpy=0 0 0
- joint shoulder_joint: origin xyz=0 0 16.35 rpy=0 0 0 -> xyz=0 0 3.7 rpy=0 0 0; parent base_rotator -> rotator
- joint twist_joint: origin xyz=0 0 14.7 rpy=0 0 0 -> xyz=0 0 7.7 rpy=0 0 0
- joint wrist_joint: limit lower=-1.57 upper=2.8 -> lower=-1.57 upper=1.57; origin xyz=0 0 15.85 rpy=0 0 0 -> xyz=0 0 12.0 rpy=0 0 0

Commit message: Inverse kinematics updates

File: code/goat_arm.urdf (robot description, URDF)
Before this commit: robot robot_arm, 7 links, 6 joints
Links:
- link base_link: geometry visual cylinder length=2 radius=1
- link fingers: geometry visual cylinder length=2 radius=2.0
- link forearm: geometry visual cylinder length=2 radius=2.0
- link hand: geometry visual cylinder length=2 radius=2.0
- link rotator: geometry visual cylinder length=2 radius=1
- link upper_arm: geometry visual cylinder length=2 radius=2.0
Joints:
- joint base_joint: origin xyz=0 0 13.3 rpy=0 0 0 -> xyz=0 0 2 rpy=0 0 0
- joint elbow_joint: origin xyz=0 0 12.0 rpy=0 0 0 -> xyz=0 0 2 rpy=0 0 0
- joint last_joint: origin xyz=0 0 7.0 rpy=0 0 0 -> xyz=0 0 2 rpy=0 0 0
- joint shoulder_joint: origin xyz=0 0 3.7 rpy=0 0 0 -> xyz=0 0 1 rpy=0 0 0
- joint twist_joint: origin xyz=0 0 7.7 rpy=0 0 0 -> xyz=0 0 2 rpy=0 0 0
- joint wrist_joint: origin xyz=0 0 12.0 rpy=0 0 0 -> xyz=0 0 2 rpy=0 0 0

Commit message: IKPY configuration

File: code/goat_arm.urdf (robot description, URDF)
Before this commit: robot robot_arm, 7 links, 6 joints
Links:
- link base_link: geometry visual cylinder length=13.5 radius=1
- link fingers: geometry visual cylinder length=13.5 radius=2.0
- link forearm: geometry visual cylinder length=12 radius=2.0
- link hand: geometry visual cylinder length=7.5 radius=2.0
- link rotator: geometry visual cylinder length=4 radius=1
- link upper_arm: geometry visual cylinder length=12.25 radius=2.0
Joints:
- joint base_joint: origin xyz=0 0 2 rpy=0 0 0 -> xyz=0 0 13.5 rpy=0 0 0
- joint elbow_joint: origin xyz=0 0 2 rpy=0 0 0 -> xyz=0 0 12.25 rpy=0 0 0
- joint last_joint: origin xyz=0 0 2 rpy=0 0 0 -> xyz=0 0 13.5 rpy=0 0 0
- joint shoulder_joint: origin xyz=0 0 1 rpy=0 0 0 -> xyz=0 0 4 rpy=0 0 0
- joint twist_joint: origin xyz=0 0 2 rpy=0 0 0 -> xyz=0 0 7.5 rpy=0 0 0
- joint wrist_joint: origin xyz=0 0 2 rpy=0 0 0 -> xyz=0 0 12 rpy=0 0 0
